Commit message: camera image stream and compression

File: scout_description/urdf/scout_description.urdf (robot description, URDF)
Before this commit: robot scout_description, 16 links, 15 joints
Links:
- added link camera_body_link, mass 0.0236867347433105; collision mesh filename=package://scout_description/meshes/camera_link.STL; visual mesh filename=package://scout_description/meshes/camera_link.STL
- link camera_link: mass 0.0236867347433105 -> None; geometry 
Joints:
- added joint camera_body_to_camera: type fixed, parent camera_body_link, child camera_link, origin xyz=0 0 0 rpy=-1.5707963267949 -1.5707963267949 0, axis 0 0 0
- joint camera_to_lens: parent camera_link -> camera_body_link
- joint mount_to_camera: child camera_link -> camera_body_link

Commit message: working LiDAR

File: scout_description/urdf/scout_description.urdf (robot description, URDF)
Before this commit: robot scout_description, 17 links, 16 joints
Links:
- added link laser
Joints:
- added joint lidar1_to_laser: type fixed, parent lidar1_link, child laser, origin xyz=0 0 0 rpy=0 1.5707963267949 1.5707963267949, axis 0 0 0
